File: MySensorsNode.sch (KiCad schematic (older format))
At the start: 45 parts, among them CON1 Opt. JST Connector, CON2 Opt. 2.5mm jack, P1 CONN_01X04, P10 CONN_01X04, P11 CONN_02X03, P2 CONN_01X04, P3 CONN_01X04, P4 CONN_01X04, P5 CONN_01X04, P6 CONN_01X04, P7 CONN_01X05, P8 CONN_01X05, P9 CONN_01X07, Q1 DMP3056L-7, Q2 DMP3056L-7, U1 TPS61097A, U2 TPS6122X, U3 RFM69HW, U4 AT25DF512C, U5 ATSHA204A, U6 NRF24L01, U7 ArduinoProMini

Commit message: Rev. 1.1 of my generic MySensors node
* Added resistor to terminate REG_BYPASS to default 'on' (fixes #2)
* Added extra RF bypass capacitors (fixes #5)
* Updated RF69 footprint to have sligtly wider space between holes
* Added optional pull-ups to CS signals on SPI devices (fixes #3)
* Reversed polarity of CON1 to fit battery default pinout (fixes #1)
* Sensor pin connector swapped in favor of MYSX 1.5 connector
* More battery options
* Discarded 5V regulator and added a different 3.3V reg for 12V input (fixes #4)
* Created layout for Superbat box BOX-2252

Things left to do:
* Update schematic with full sourcing details
* Create 5x5cm layout (default)
* Create Superbat box LE-BOX-0028 layout
* Create manufacturing outputs
* Create BOM(s)
Parts:
- removed C3, C4, C6: 10uF, Capacitors_SMD:C_1206_HandSoldering, symbol C
- removed CON1: Opt. JST Connector, w_conn_jst-ph:s2b-ph-kl, symbol CONN_01X02
- removed CON2: Opt. 2.5mm jack, w_conn_misc:dc_socket, symbol JACK_2P
- removed L2: 4.7uH, Capacitors_SMD:C_0805_HandSoldering, symbol INDUCTOR
- removed P1, P10, P2, P3, P4, P5, P6: CONN_01X04, Pin_Headers:Pin_Header_Straight_1x04, symbol CONN_01X04
- removed P7, P8: CONN_01X05, Pin_Headers:Pin_Header_Straight_1x05, symbol CONN_01X05
- removed P9: CONN_01X07, Pin_Headers:Pin_Header_Straight_1x07, symbol CONN_01X07
- removed R4: 1M, Resistors_SMD:R_0805_HandSoldering, symbol R
- removed U2: TPS6122X, Housings_SOT-23_SOT-143_TSOT-6:SC-70-6_Handsoldering, symbol TPS6122X
- added BT1: 2.5mm jack, mysensors_connectors:dc_socket-kcswalter, symbol JACK_2P
- added BT2: JST, mysensors_connectors:s2b-ph-kl-kcswalter, symbol Battery
- added BT3: Generic, mysensors_connectors:TerminalBlock2.54mmx2-kcswalter, symbol Battery
- added BT4: CR123, mysensors_connectors:CR123_holder, symbol Battery
- added BT5: 24.5mm, mysensors_connectors:keystone_3009-kcswalter, symbol Battery
- added C1: 47uF, Capacitors_Tantalum_SMD:TantalC_SizeC_EIA-6032_HandSoldering, symbol CP
- added C10, C12, C13, C14, C2: 4.7uF, Capacitors_Tantalum_SMD:TantalC_SizeB_EIA-3528_HandSoldering, symbol CP
- added C15, C16, C18, C7: 0.1uF, Capacitors_SMD:C_1206_HandSoldering, symbol C
- added C3, C4: 10uF, Capacitors_Tantalum_SMD:TantalC_SizeA_EIA-3216_HandSoldering, symbol CP
- added C8: C, Resistors_Universal:Resistor_SMD+THTuniversal_0805to1206_RM10_HandSoldering, symbol C
- added JP10, JP6, JP7: Jumper_NO_Small, Pin_Headers:Pin_Header_Straight_1x02, symbol Jumper_NO_Small
- added JP2: JUMPER3, Pin_Headers:Pin_Header_Straight_1x03, symbol JUMPER3
- added P1: MYSX_1.5, mysensors_connectors:MYSX_1.5, symbol MYSX_1.5
- added P3, P4: CONN_01X03, Pin_Headers:Pin_Header_Straight_1x03, symbol CONN_01X03
- added R6, R7, R8, R9: 56K, Resistors_SMD:R_0805_HandSoldering, symbol R
- added RV1: 1M, Potentiometers:Potentiometer_Bourns_3296Y_3-8Zoll_Angular_ScrewUp, symbol POT
- added U1: LD1117DT33TR, SMD_Packages:DPAK-2, symbol LD1117S33TR
- added U8: Si7021, Housings_DFN_QFN:DFN-6-1EP_3x3mm_Pitch0.95mm, symbol Si7021
- L1: Supplier1 link http://www.mouser.com/ProductDetail/Taiyo-Yuden/CBC2012T4R7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 -> http://se.mouser.com/ProductDetail/Taiyo-Yuden/CBC2012T4R7M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; Supplier2 link http://se.farnell.com/tdk/mlz2012m4r7wt/inductor-shielded-4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 -> (none); Supplier2 part 2215656 -> (none); Supplier4 link http://www.digikey.se/short/7w1zf0 -> http://www.digikey.se/short/tc5dd3; Supplier4 part 587-2527-1-ND -> 587-1602-1-ND; Vendor TDK -> Taiyo Yuden; Vendor part MLZ2012M4R7WT -> CBC2012T4R7M
- R1: value 402K -> 150K; Supplier1 link http://se.mouser.com/ProductDetail/Welwyn-Components-TT-Ele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 -> http://se.mouser.com/ProductDetail/Vishay-Dale/CRCW0805150K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; Supplier1 part 756-PCF0805R-402KBT1 -> 71-CRCW0805-150K-E3; Supplier2 link http://se.farnell.com/te-connectivity/rp73pf2a402kbtdf/mots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 -> http://se.farnell.com/welwyn/pcf0805r-150kbt1/resistor-0805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; Supplier2 part 2117439RL -> 1160270RL; Supplier3 link https://www.elfa.se/elfa3~se_en/elfa/init.do?item=10-525-18 -> https://www.elfa.se/elfa3~se_sv/elfa/init.do?item=60-587-70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; Supplier3 part 10-525-18 -> 60-587-70; Supplier4 link http://www.digikey.com/short/7dmdrq -> http://www.digikey.se/short/tcbcn3; Supplier4 part 985-1359-1-ND -> 541-150KCCT-ND; Vendor Welwyn Components / TT Electronics -> Vishay / Dale; Vendor part PCF0805R-402KBT1 -> CRCW0805150KFKEA
- U7: footprint mysensors_arduino:pro_mini_china -> mysensors_arduino:pro_mini
- renumbered C7 to C11, C8 to C17, C2 to C5, C1 to C6, C5 to C9, JP4 to JP1, JP2 to JP3, JP1 to JP4, JP3 to JP5, JP5 to JP8, JP6 to JP9, P11 to P2, R5 to R4, R6 to R5, U1 to U2, U5 to U3, U3 to U4, U6 to U5, U4 to U6
Connections:
- net labels added: ATSHA_SDA, MYSX_3.3V_EN, MYSX_A1, MYSX_A2, MYSX_D10_A4, MYSX_D14_CS, MYSX_D1_DFM, MYSX_D2_DTM, MYSX_D3_INT, MYSX_D4_INT, MYSX_D5_PWM, MYSX_D6_PWM, MYSX_D7_SCL, MYSX_D8_SDA, MYSX_D9_A3
- net labels removed: +5P, ASENS0, ASENS1, DSENS0_URX, DSENS1_UTX, DSENS2_PWM, I2C_SCL, I2C_SDA, INT1, INT2, REG_BYPASS, SENSOR_EN, SPI_CSN, VBAT_SMPL_EN
- wire segments 104 -> 102
- no-connect marks 9 -> 8
Other:
- note added: "3.3V power management"
- note added: "Adjust RV1 depending on\nADC resolution, reference\nvoltage and input voltage"
- note added: "Battery measurement"
- note added: "High voltage LDO regulation (max 12V input voltage)"
- note added: "I2C Pulls"
- note added: "JP1 and JP7 serves as current measurement taps. They have to be shorted in order to provide board power.\nJP1 for onboard power and JP7 for daughter board power."
- note added: "JP1 is a current measurement tap\nIt must be shorted for proper board use"
- note added: "JP10 enables MYSX_D9_A3 to be used to take a low-power battery sample.\nAnalog samples from a daughterboard might not work well in this case."
- note added: "JP2 is used to select either high voltage regulation or low voltage regulation for 3.3V rail.\nPos 1-2 selects low-voltage and pos 2-3 selects high-voltage."
- note added: "JP3 bypasses 3.3V regulator to connect battery directly to 3.3V net."
- note added: "JP4 bypasses low-power battery sampling circuitry in favor of "default" voltage divider mechanism.\nLow-power battery sampling is activated by driving MYSX_D9_A3 low together with JP10."
- note added: "JP5 bypasses sensor power switch to permanently supply 3.3V to MYSX connector,\nelse rail is enabled by driving MYSX_3.3V_EN low."
- note added: "JP6 enables MYSX_D10_A4 to be used to bypass low-voltage regulator\n(when battery voltage is in an acceptable region to be used directly)."
- note added: "JP7 is a current measurement tap\nIt must be shorted for daughter board use"
- note added: "JP8 selects INT1 interrupt source. Pos 1-2 selects MYSX_D3_INT source and pos 2-3 selects RF board."
- note added: "JP9 selects SPI SS destination. Pos 1-2 selects RF24 and pos 2-3 selects RF69."
- note added: "Larger capacitor value gives a larger sampling\nwindow"
- note added: "Low voltage step-up regulation (max 4.2V input voltage)"
- note added: "MYSX connector"
- note added: "Optional"
- note added: "Optional MYSX 3.3V power toggle"
- note added: "Optional components for\nlow-power sampling:\nQ1,R2,C9"
- note added: "Optional components for\nlow-power sampling:\nR3, Q2"
- note added: "Optional decouplung for\nmeasurement stability"
- note added: "Power connectors (no need to mount them all unless desired)"
- note added: "Regulator bypass"
- note added: "Regulator selection"
- note added: "Sensor power rails"
- note added: "Short JP1 to enable continous\nVBAT_SMPL values"
- note added: "Short JP10 to enable\nlow-power battery sampling"
- note added: "Short JP5 to bypass MCU\ncontrolled MYSX 3.3V rail"
- note added: "Short JP6 to enable MCU controlled bypass of regulator"
- note added: "Temp/hum sensor"
- note removed: "Header layout"
- note removed: "JP1 bypasses low-power battery sampling circuitry in\nfavor of "default" voltage divider mechanism."
- note removed: "JP2 bypasses 3.3V regulator to connect battery directly\nto 3.3V net."
- note removed: "JP3 bypasses sensor power switch to permanently supply\n3.3V and 5V sensor power rail."
- note removed: "JP4 is just used for power measurement and should\nnormally be shorted."
- note removed: "JP5 selects INT1 interrupt source. Pos 1-2 selects INT1\nsource on P10 and pos 2-3 selects RF board."
- note removed: "JP6 selects SPI SS destination. Pos 1-2 selects RF24\nand pos 2-3 selects RF69."
- note removed: "Power connectors"
- note removed: "Power management"
- note removed: "Px:1 -> 5V\nPx:2 -> 3.3V\nPx:3 -> GND\nP1:4 -> D1 (UART TX)\nP2:4 -> D0 (UART RX)\nP3:4 -> D3 (INT2)\nP4:4 -> D6 (PWM)\nP5:4 -> A7\nP6:4 -> A6\nP7:4 -> A4 (I2C SDA)\nP7:5 -> A5 (I2C SCL)\nP8:4 -> A4 (I2C SDA)\nP8:5 -> A5 (I2C SCL)\nP9:4 -> MISO\nP9:5 -> MOSI\nP9:6 -> SCK\nP9:7 -> D7 (SPI_CSn)"
- moved on the sheet: ANT1, C11, C17, C5, C6, C9, JP1, JP3, JP4, JP5, JP8, JP9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

Commit message: Minor beautifications and updated CHANGES.txt
Changed lines of the file:
@@
 07 00 85 88 3B 00 28 44 DC 01 40 21 E2 0E 00 0A 11 77 00 50 88 B8 03 80 42 C4 1D 00 14 22 EE 00
 A0 10 71 07 00 85 88 3B 00 28 F4 2F 6E 0E 73 66 69 F5 31 42 00 00 00 00 49 45 4E 44 AE 42 60 82
-B8
+B1
 EndData
 $EndBitmap
@@
 MISO
 Entry Wire Line
-	6600 4500 6700 4600
-Entry Wire Line
-	5850 4500 5950 4600
-Entry Wire Line
-	5750 4500 5850 4600
+	6500 4600 6600 4500
+Entry Wire Line
+	5750 4600 5850 4500
+Entry Wire Line
+	5650 4600 5750 4500
 $Comp
 L GND #PWR024

Commit message: Updated U1 footprint
U1 footprint is now available in the mysensors-kicad repository
Parts:
- U1: footprint SMD_Packages:DPAK-2 -> mysensors_obscurities:d-pak-kcswalter
Changed lines of the file:
@@
 $Bitmap
 Pos 10350 6850
-Scale 1.000000
+Scale 1,000000
 Data
 89 50 4E 47 0D 0A 1A 0A 00 00 00 0D 49 48 44 52 00 00 01 F4 00 00 00 AC 08 02 00 00 00 02 1E C9
@@
 07 00 85 88 3B 00 28 44 DC 01 40 21 E2 0E 00 0A 11 77 00 50 88 B8 03 80 42 C4 1D 00 14 22 EE 00
 A0 10 71 07 00 85 88 3B 00 28 F4 2F 6E 0E 73 66 69 F5 31 42 00 00 00 00 49 45 4E 44 AE 42 60 82
-B1
+30
 EndData
 $EndBitmap
@@
 $Bitmap
 Pos 9250 6850
-Scale 1.000000
+Scale 1,000000
 Data
 89 50 4E 47 0D 0A 1A 0A 00 00 00 0D 49 48 44 52 00 00 00 A8 00 00 00 70 08 02 00 00 00 05 44 AC
@@
 F 0 "U1" H 5300 1250 40  0000 C CNN
 F 1 "LD1117DT33TR" H 5100 1150 40  0000 C CNN
-F 2 "SMD_Packages:DPAK-2" H 5100 1150 40  0001 C CNN
+F 2 "mysensors_obscurities:d-pak-kcswalter" H 5100 1150 40  0001 C CNN
 F 3 "http://www.st.com/st-web-ui/static/active/en/resource/technical/document/datasheet/CD00000544.pdf" H 5100 1050 60  0001 C CNN
 F 4 "STMicroelectronics" H 5100 1050 60  0001 C CNN "Vendor"

Commit message: Added a step-up reg and some sourcing details
Added TI TPS61221 (3.3V fixed) as an alternative to TPS61097A.
Also added some more sourcing details to some components in the
schematic.
Parts:
- added U9: TPS6122X, Housings_SOT-23_SOT-143_TSOT-6:SC-70-6, symbol TPS6122X
- BT1: Supplier5 (none) -> AliExpress; Supplier5 link (none) -> http://www.aliexpress.com/item/2-5mm-DC-Jack-DC-Socket-DC-P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; Supplier5 part (none) -> 1614043178
- BT2: Supplier5 (none) -> AliExpress; Supplier5 link (none) -> http://www.aliexpress.com/item/free-shipping-2-0mm-2pin-hea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; Supplier5 part (none) -> 1709786094
- BT3: Supplier1 (none) -> Mouser; Supplier1 link (none) -> http://www.mouser.se/ProductDetail/TE-Connectivity/282834-2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; Supplier1 part (none) -> 571-282834-2; Supplier2 (none) -> Digi-Key; Supplier2 link (none) -> http://www.digikey.com/short/tzt88w; Supplier2 part (none) -> ED10561-ND; Supplier5 (none) -> AliExpress; Supplier5 link (none) -> http://www.aliexpress.com/item/20pcs-2-Poles-2-Pin-2-54mm-0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; Supplier5 part (none) -> 1252981306; Vendor (none) -> TE Connectivity; Vendor part (none) -> 282834-2
- BT4: Supplier1 link (none) -> http://www.ebay.com/itm/181790677824; Supplier1 part (none) -> 181790677824
- Q1, Q2: Supplier5 (none) -> AliExpress; Supplier5 link (none) -> http://www.aliexpress.com/item/Free-Shipping-20PCS-lot-DMP3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; Supplier5 part (none) -> 32446073237
- U1: Supplier4 Digi-Key -> (none); Supplier5 (none) -> AliExpress; Supplier5 link (none) -> http://www.aliexpress.com/item/ICIC-LD1117-LD1117DT33TR-LD1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; Supplier5 part (none) -> 32395965284
- U7: Supplier5 (none) -> AliExpress; Supplier5 link (none) -> http://www.aliexpress.com/item/1pcs-lot-Pro-Mini-328-Mini-3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; Supplier5 part (none) -> 32313595044
Connections:
- wire segments 102 -> 140
Other:
- note added: "NOTE: U2 and U9 are mutually exclusive"
- moved on the sheet: C5, C6, JP6, L1, R1, U2

Commit message: Added more sourcing details
Also minor schematic beautifications
Parts:
- BT1: Supplier1 Mouser -> AliExpress; Supplier1 link http://www.mouser.com/ProductDetail/Switchcraft/RAPC712X/?q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 -> http://www.aliexpress.com/item/2-5mm-DC-Jack-DC-Socket-DC-P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; Supplier1 part 502-RAPC712X -> 1614043178; Supplier2 Farnell -> Digi-Key; Supplier2 link http://se.farnell.com/switchcraft/rapc712x/jack-socket-dc-2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 -> http://www.digikey.se/short/7wd85d; Supplier2 part 1608726 -> CP-037B-ND; Supplier3 Elfa -> Mouser; Supplier3 link https://www.elfa.se/elfa3~se_en/elfa/init.do?item=42-205-20 -> http://www.mouser.com/ProductDetail/Switchcraft/RAPC712X/?q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; Supplier3 part 42-205-20 -> 502-RAPC712X; Supplier4 Digi-Key -> Farnell; Supplier4 link http://www.digikey.se/short/7wd85d -> http://se.farnell.com/switchcraft/rapc712x/jack-socket-dc-2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; Supplier4 part CP-037B-ND -> 1608726; Supplier5 AliExpress -> Elfa; Supplier5 link http://www.aliexpress.com/item/2-5mm-DC-Jack-DC-Socket-DC-P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 -> https://www.elfa.se/elfa3~se_en/elfa/init.do?item=42-205-20; Supplier5 part 1614043178 -> 42-205-20
- BT2: Supplier1 Electrokit Sweden AB -> AliExpress; Supplier1 link http://www.electrokit.com/stiftlist-ph-2pol-2-0mm-vinklad.5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 -> http://www.aliexpress.com/item/free-shipping-2-0mm-2pin-hea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; Supplier1 part 41012805 -> 1709786094; Supplier3 Elfa -> Digi-Key; Supplier3 link https://www.elfa.se/elfa3~se_en/elfa/init.do?item=43-019-56 -> http://www.digikey.se/short/7wd8fm; Supplier3 part 43-019-56 -> 455-1719-ND; Supplier4 Digi-Key -> Electrokit Sweden AB; Supplier4 link http://www.digikey.se/short/7wd8fm -> http://www.electrokit.com/stiftlist-ph-2pol-2-0mm-vinklad.5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; Supplier4 part 455-1719-ND -> 41012805; Supplier5 AliExpress -> Elfa; Supplier5 link http://www.aliexpress.com/item/free-shipping-2-0mm-2pin-hea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 -> https://www.elfa.se/elfa3~se_en/elfa/init.do?item=43-019-56; Supplier5 part 1709786094 -> 43-019-56
- BT3: Supplier1 Mouser -> AliExpress; Supplier1 link http://www.mouser.se/ProductDetail/TE-Connectivity/282834-2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 -> http://www.aliexpress.com/item/20pcs-2-Poles-2-Pin-2-54mm-0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; Supplier1 part 571-282834-2 -> 1252981306; Supplier3 (none) -> Mouser; Supplier3 link (none) -> http://www.mouser.se/ProductDetail/TE-Connectivity/282834-2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; Supplier3 part (none) -> 571-282834-2; Supplier5 AliExpress -> (none); Supplier5 link http://www.aliexpress.com/item/20pcs-2-Poles-2-Pin-2-54mm-0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 -> (none); Supplier5 part 1252981306 -> (none)
- C1: Supplier1 Mouser -> AliExpress; Supplier1 link http://se.mouser.com/ProductDetail/AVX/TPSC476K016R0350/?qs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 -> http://www.aliexpress.com/item/Free-Shipping-6032-SMD-Tanta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; Supplier1 part 581-TPSC476K016R0350 -> 32444935172; Supplier2 Farnell -> Digi-Key; Supplier2 link http://se.farnell.com/vishay-sprague/tr3c476k016c0350/cap-t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 -> http://www.digikey.se/short/t3t5v5; Supplier2 part 1754090 -> 478-1773-1-ND; Supplier3 Digi-Key -> Mouser; Supplier3 link http://www.digikey.se/short/t3t5v5 -> http://se.mouser.com/ProductDetail/AVX/TPSC476K016R0350/?qs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; Supplier3 part 478-1773-1-ND -> 581-TPSC476K016R0350; Supplier4 (none) -> Farnell; Supplier4 link (none) -> http://se.farnell.com/vishay-sprague/tr3c476k016c0350/cap-t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; Supplier4 part (none) -> 1754090
- C10, C12, C13, C14: Supplier2 link (none) -> http://se.farnell.com/avx/tpsb475k025r0900/cap-tant-4-7uf-2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; Supplier2 part (none) -> 1432589RL; Supplier4 (none) -> Elfa; Supplier4 link (none) -> https://www.elfa.se/elfa3~se_sv/elfa/init.do?item=67-700-69; Supplier4 part (none) -> 67-700-69; Supplier5 (none) -> AliExpress; Supplier5 link (none) -> http://www.aliexpress.com/item/Free-shipping-20pcs-B-3528-4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; Supplier5 part (none) -> 32456411946
- C11, C15, C16, C17, C18, C7: Supplier1 Mouser -> Farnell; Supplier1 link http://se.mouser.com/ProductDetail/Vishay-Vitramon/VJ1206Y1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 -> http://se.farnell.com/multicomp/mcsh31b104k250ct/cap-mlcc-x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; Supplier1 part 77-VJ1206Y104KXQPBC -> 1856619; Supplier2 Farnell -> Mouser; Supplier2 link http://se.farnell.com/multicomp/mcsh31b104k250ct/cap-mlcc-x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 -> http://se.mouser.com/ProductDetail/Vishay-Vitramon/VJ1206Y1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; Supplier2 part 1856619 -> 77-VJ1206Y104KXQPBC; Supplier3 Elfa -> Digi-Key; Supplier3 link https://www.elfa.se/elfa3~se_en/elfa/init.do?item=65-724-45 -> http://www.digikey.se/short/7w1zrd; Supplier3 part 65-724-45 -> 399-1249-1-ND; Supplier4 Digi-Key -> AliExpress; Supplier4 link http://www.digikey.se/short/7w1zrd -> http://www.aliexpress.com/item/1206-100NF-104M-Y5V-50V-SMD-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; Supplier4 part 399-1249-1-ND -> 32274650296; Supplier5 (none) -> Elfa; Supplier5 link (none) -> https://www.elfa.se/elfa3~se_en/elfa/init.do?item=65-724-45; Supplier5 part (none) -> 65-724-45
- C2: Supplier1 Mouser -> AliExpress; Supplier1 link http://se.mouser.com/ProductDetail/AVX/TPSB475K025R0900/?qs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 -> http://www.aliexpress.com/item/Free-shipping-20pcs-B-3528-4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; Supplier1 part 581-TPSB475K025R0900 -> 32456411946; Supplier2 link (none) -> http://se.farnell.com/avx/tpsb475k025r0900/cap-tant-4-7uf-2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; Supplier2 part (none) -> 1432589RL; Supplier4 (none) -> Mouser; Supplier4 link (none) -> http://se.mouser.com/ProductDetail/AVX/TPSB475K025R0900/?qs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; Supplier4 part (none) -> 581-TPSB475K025R0900; Supplier5 (none) -> Elfa; Supplier5 link (none) -> https://www.elfa.se/elfa3~se_sv/elfa/init.do?item=67-700-69; Supplier5 part (none) -> 67-700-69
- C3, C4: Supplier1 link http://se.mouser.com/ProductDetail/AVX/F930J476MAA/?qs=sGAE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 -> http://www.mouser.se/ProductDetail/AVX/F931C106MAA/?qs=sGAE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; Supplier1 part 647-F930J476MAA -> 647-F931C106MAA; Supplier2 link http://se.farnell.com/kemet/t494a476m006at/tantalum-capacit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 -> http://se.farnell.com/vishay-sprague/tp3a106k016c1700as/cap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; Supplier2 part 1639991 -> 2493378; Supplier3 Elfa -> Digi-Key; Supplier3 link https://www.elfa.se/elfa3~se_sv/elfa/init.do?item=67-707-88 -> http://www.digikey.se/short/t4q4zv; Supplier3 part 67-707-88 -> 478-8237-1-ND; Supplier4 Digi-Key -> (none); Supplier4 link http://www.digikey.se/short/ttj883 -> (none); Supplier4 part 478-8180-1-ND -> (none); Vendor part F930J476MAA -> F931C106MAA
- C5, C6: Supplier1 Mouser -> AliExpress; Supplier1 link http://se.mouser.com/Search/ProductDetail.aspx?R=VJ1206V106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 -> http://www.aliexpress.com/item/100pcs-1206-3216-106K-10uF-1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; Supplier1 part 77-VJ1206V106ZXQTBC -> 32308484869; Supplier2 Farnell -> Mouser; Supplier2 link http://se.farnell.com/multicomp/mc1206f106z100ct/cap-mlcc-y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 -> http://se.mouser.com/Search/ProductDetail.aspx?R=VJ1206V106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; Supplier2 part 1759434 -> 77-VJ1206V106ZXQTBC; Supplier3 Elfa -> Farnell; Supplier3 link https://www.elfa.se/elfa3~se_en/elfa/init.do?item=65-721-38 -> http://se.farnell.com/multicomp/mc1206f106z100ct/cap-mlcc-y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; Supplier3 part 65-721-38 -> 1759434; Supplier5 (none) -> Elfa; Supplier5 link (none) -> https://www.elfa.se/elfa3~se_en/elfa/init.do?item=65-721-38; Supplier5 part (none) -> 65-721-38
- C8: Supplier5 (none) -> AliExpress
- C9: Supplier1 link http://se.mouser.com/ProductDetail/Vishay-Vitramon/VJ1206Y1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 -> http://www.mouser.se/ProductDetail/Vishay-Vitramon/VJ1206Y1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; Supplier1 part 77-VJ1206Y104KXQPBC -> 77-VJ1206Y104KXXCBC; Supplier2 link http://se.farnell.com/multicomp/mcsh31b104k250ct/cap-mlcc-x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 -> http://se.farnell.com/multicomp/mc1206b104k250ct/cap-mlcc-x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; Supplier2 part 1856619 -> 1759312; Supplier3 Elfa -> Digi-Key; Supplier3 link https://www.elfa.se/elfa3~se_en/elfa/init.do?item=65-724-45 -> http://www.digikey.se/short/t4zm2w; Supplier3 part 65-724-45 -> 1276-2742-1-ND; Supplier4 Digi-Key -> Elfa; Supplier4 link http://www.digikey.se/short/7w1zrd -> https://www.elfa.se/elfa3~se_en/elfa/init.do?item=65-722-69; Supplier4 part 399-1249-1-ND -> 65-722-69; Supplier5 (none) -> AliExpress; Supplier5 link (none) -> http://www.aliexpress.com/item/200pcs-lot-CL31B104KACNNNC-C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; Supplier5 part (none) -> 32323646062; Vendor MULTICOMP -> Vishay; Vendor part RR1220P-105-B-T5 -> VJ1206Y104KXXCW1BC
- JP1, JP3, JP6: Supplier1 Mouser -> Farnell; Supplier1 link http://www.mouser.com/ProductDetail/Wurth-Electronics/61300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 -> http://se.farnell.com/wurth-elektronik/61300211121/header-2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; Supplier1 part 710-61300211121 -> 2356153; Supplier2 Farnell -> Digi-Key; Supplier2 link http://se.farnell.com/wurth-elektronik/61300211121/header-2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 -> http://www.digikey.se/short/7w149z; Supplier2 part 2356153 -> S1012EC-02-ND; Supplier3 Elfa -> Mouser; Supplier3 link https://www.elfa.se/elfa3~se_en/elfa/init.do?item=43-004-90 -> http://www.mouser.com/ProductDetail/Wurth-Electronics/61300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; Supplier3 part 43-004-90 -> 710-61300211121; Supplier4 Digi-Key -> Elfa; Supplier4 link http://www.digikey.se/short/7w149z -> https://www.elfa.se/elfa3~se_en/elfa/init.do?item=43-004-90; Supplier4 part S1012EC-02-ND -> 43-004-90
- JP2, JP8, JP9: Supplier1 Mouser -> Farnell; Supplier1 link http://www.mouser.com/ProductDetail/3M-Electronic-Solutions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 -> http://se.farnell.com/multicomp/2211s-03g/header-1-row-vert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; Supplier1 part 517-9611036804AR -> 1593412; Supplier2 Farnell -> Digi-Key; Supplier2 link http://se.farnell.com/multicomp/2211s-03g/header-1-row-vert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 -> http://www.digikey.se/short/7w1485; Supplier2 part 1593412 -> 952-2264-ND; Supplier3 Elfa -> Mouser; Supplier3 link https://www.elfa.se/elfa3~se_en/elfa/init.do?item=43-004-91 -> http://www.mouser.com/ProductDetail/3M-Electronic-Solutions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; Supplier3 part 43-004-91 -> 517-9611036804AR; Supplier4 Digi-Key -> Elfa; Supplier4 link http://www.digikey.se/short/7w1485 -> https://www.elfa.se/elfa3~se_en/elfa/init.do?item=43-004-91; Supplier4 part 952-2264-ND -> 43-004-91
- L1: Supplier1 Mouser -> Farnell; Supplier1 link http://se.mouser.com/ProductDetail/Taiyo-Yuden/CBC2012T4R7M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 -> http://se.farnell.com/tdk/mlz2012m4r7wt/inductor-shielded-4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; Supplier1 part 963-CBC2012T4R7M -> 2215656; Supplier2 Farnell -> Digi-Key; Supplier2 link (none) -> http://www.digikey.se/short/tc5dd3; Supplier2 part (none) -> 587-1602-1-ND; Supplier3 Elfa -> Mouser; Supplier3 link https://www.elfa.se/elfa3~se_en/elfa/init.do?item=10-969-35 -> http://se.mouser.com/ProductDetail/Taiyo-Yuden/CBC2012T4R7M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; Supplier3 part 10-969-35 -> 963-CBC2012T4R7M; Supplier4 Digi-Key -> Elfa; Supplier4 link http://www.digikey.se/short/tc5dd3 -> https://www.elfa.se/elfa3~se_en/elfa/init.do?item=10-969-35; Supplier4 part 587-1602-1-ND -> 10-969-35
- P1: Supplier1 (none) -> Elfa; Supplier1 link (none) -> https://www.elfa.se/elfa3~se_en/elfa/init.do?item=43-702-35; Supplier1 part (none) -> 43-702-35; Supplier2 (none) -> Mouser; Supplier2 link (none) -> http://www.mouser.se/ProductDetail/Harwin/M20-9981045/?qs=%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; Supplier2 part (none) -> 855-M20-9981045; Supplier3 (none) -> Digi-Key; Supplier3 link (none) -> http://www.digikey.se/short/t4z5r3; Supplier3 part (none) -> 952-2129-ND; Supplier4 (none) -> Farnell; Supplier4 link (none) -> http://se.farnell.com/harwin/m20-9981045/board-to-board-con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; Supplier4 part (none) -> 2127560; Vendor (none) -> HARWIN; Vendor part (none) -> M20-9981045
- P2: Supplier1 link http://www.mouser.com/ProductDetail/TE-Connectivity/5-14625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 -> http://www.mouser.se/ProductDetail/Harwin/M20-9981045/?qs=%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; Supplier1 part 571-5-146252-3 -> 855-M20-9981045; Supplier2 link http://se.farnell.com/harwin/m20-9980345/header-tht-vertica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 -> http://se.farnell.com/harwin/m20-9981045/board-to-board-con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; Supplier2 part 1022230 -> 2127560; Vendor part M20-9980345 -> M20-9981045
- P3, P4: Supplier1 (none) -> Farnell; Supplier1 link (none) -> http://se.farnell.com/multicomp/2211s-03g/header-1-row-vert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; Supplier1 part (none) -> 1593412; Supplier2 (none) -> Digi-Key; Supplier2 link (none) -> http://www.digikey.se/short/7w1485; Supplier2 part (none) -> 952-2264-ND; Supplier3 (none) -> Mouser; Supplier3 link (none) -> http://www.mouser.com/ProductDetail/3M-Electronic-Solutions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; Supplier3 part (none) -> 517-9611036804AR; Supplier4 (none) -> Elfa; Supplier4 link (none) -> https://www.elfa.se/elfa3~se_en/elfa/init.do?item=43-004-91; Supplier4 part (none) -> 43-004-91; Vendor (none) -> HARWIN; Vendor part (none) -> M20-9993646
- Q1, Q2: Supplier1 Mouser -> AliExpress; Supplier1 link http://www.mouser.com/ProductDetail/Diodes-Incorporated/DMP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 -> http://www.aliexpress.com/item/Free-Shipping-20PCS-lot-DMP3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; Supplier1 part 621-DMP3056L-7 -> 32446073237; Supplier2 Farnell -> Mouser; Supplier2 link http://se.farnell.com/nxp/pmv32up/mosfet-p-ch-20v-4a-sot23/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 -> http://www.mouser.com/ProductDetail/Diodes-Incorporated/DMP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; Supplier2 part 1894624 -> 621-DMP3056L-7; Supplier3 Elfa -> Digi-Key; Supplier3 link https://www.elfa.se/elfa3~se_en/elfa/init.do?item=71-397-02 -> http://www.digikey.se/short/7wd8q3; Supplier3 part 71-397-02 -> DMP3056L-7DICT-ND; Supplier4 Digi-Key -> Elfa; Supplier4 link http://www.digikey.se/short/7wd8q3 -> https://www.elfa.se/elfa3~se_en/elfa/init.do?item=71-397-02; Supplier4 part DMP3056L-7DICT-ND -> 71-397-02; Supplier5 AliExpress -> Farnell; Supplier5 link http://www.aliexpress.com/item/Free-Shipping-20PCS-lot-DMP3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 -> http://se.farnell.com/nxp/pmv32up/mosfet-p-ch-20v-4a-sot23/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; Supplier5 part 32446073237 -> 1894624
- R1: Supplier1 Mouser -> AliExpress; Supplier1 link http://se.mouser.com/ProductDetail/Vishay-Dale/CRCW0805150K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 -> http://www.aliexpress.com/item/0805-SMD-Resistors-150K-150K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; Supplier1 part 71-CRCW0805-150K-E3 -> 32218540982; Supplier3 Elfa -> Mouser; Supplier3 link https://www.elfa.se/elfa3~se_sv/elfa/init.do?item=60-587-70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 -> http://se.mouser.com/ProductDetail/Vishay-Dale/CRCW0805150K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; Supplier3 part 60-587-70 -> 71-CRCW0805-150K-E3; Supplier5 (none) -> Elfa; Supplier5 link (none) -> https://www.elfa.se/elfa3~se_sv/elfa/init.do?item=60-587-70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; Supplier5 part (none) -> 60-587-70
- R2, R3, R4, R5: Supplier1 Mouser -> AliExpress; Supplier1 link http://se.mouser.com/Search/ProductDetail.aspx?R=RR1220P-10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 -> http://www.aliexpress.com/item/1000-PCS-0805-10K-103-1-SMD-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; Supplier1 part 754-RR1220P-103D -> 681263963; Supplier2 Farnell -> Mouser; Supplier2 link http://se.farnell.com/susumu/rr1220p-103-d/tunnfilm-chipmot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 -> http://se.mouser.com/Search/ProductDetail.aspx?R=RR1220P-10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; Supplier2 part 1653284 -> 754-RR1220P-103D; Supplier4 Digi-Key -> Farnell; Supplier4 link http://www.digikey.se/short/7wv3tf -> http://se.farnell.com/susumu/rr1220p-103-d/tunnfilm-chipmot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; Supplier4 part RR12P10.0KDCT-ND -> 1653284; Supplier5 (none) -> Digi-Key; Supplier5 link (none) -> http://www.digikey.se/short/7wv3tf; Supplier5 part (none) -> RR12P10.0KDCT-ND
- R6, R7, R8, R9: Supplier1 Mouser -> AliExpress; Supplier1 link http://se.mouser.com/ProductDetail/Susumu/RR1220P-563-D/?qs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 -> http://www.aliexpress.com/item/0805-SMD-Resistors-56K-56K-o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; Supplier1 part 754-RR1220P-563D -> 32218601304; Supplier2 Farnell -> Mouser; Supplier2 link http://se.farnell.com/yageo-phycomp/rt0603fre0756kl/motst-n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 -> http://se.mouser.com/ProductDetail/Susumu/RR1220P-563-D/?qs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; Supplier2 part 1500644RL -> 754-RR1220P-563D; Supplier3 Elfa -> Farnell; Supplier3 link https://www.elfa.se/elfa3~se_en/elfa/init.do?item=60-255-52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 -> http://se.farnell.com/yageo-phycomp/rt0603fre0756kl/motst-n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; Supplier3 part 60-255-52 -> 1500644RL; Supplier4 Digi-Key -> Elfa; Supplier4 link http://www.digikey.se/short/7v5tfw -> https://www.elfa.se/elfa3~se_en/elfa/init.do?item=60-255-52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; Supplier4 part 541-56KACT-ND -> 60-255-52; Supplier5 (none) -> Digi-Key; Supplier5 link (none) -> http://www.digikey.se/short/7v5tfw; Supplier5 part (none) -> 541-56KACT-ND
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Connections:
- wire segments 140 -> 108
Other:
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
Commit message: Completed sourcing details of all components
Sourcing data is organized in the following way:
Supplier1 - The primary supplier (also the cheapest)
Supplier1 part - The primary supplier part number
Supplier1 link - Link to the part on the suppliers homepage

The same goes for Supplier2 to 5.
All parts also have a Vendor and Vendor part field to identify
a vendor for each part.

Fixes #6
Parts:
- BT1: Supplier5 Elfa -> RS; Supplier5 link https://www.elfa.se/elfa3~se_en/elfa/init.do?item=42-205-20 -> http://se.rs-online.com/web/p/dc-power-plugs/8786724; Supplier5 part 42-205-20 -> 878-6724
- BT2: Supplier4 Electrokit Sweden AB -> RS; Supplier4 link http://www.electrokit.com/stiftlist-ph-2pol-2-0mm-vinklad.5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 -> http://se.rs-online.com/web/p/pcb-headers/8201494; Supplier4 part 41012805 -> 820-1494
- BT4: Supplier1 E-Bay -> eBay; Supplier2 (none) -> AliExpress; Supplier2 link (none) -> http://www.aliexpress.com/item/20PCS-LOT-Plastic-Battery-Ho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; Supplier2 part (none) -> 724661148; Supplier3 (none) -> Digi-Key; Supplier3 link (none) -> http://www.digikey.se/short/t4b3bp; Supplier3 part (none) -> 36-1051-ND; Supplier4 (none) -> Mouser; Supplier4 link (none) -> http://www.mouser.se/ProductDetail/Keystone-Electronics/105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; Supplier4 part (none) -> 534-1051; Vendor (none) -> Keystone Electronics; Vendor part (none) -> 1051
- BT5: Supplier1 Mouser -> Digi-Key; Supplier1 link http://se.mouser.com/ProductDetail/Keystone-Electronics/303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 -> http://www.digikey.se/short/t4bqwf; Supplier1 part 534-3039 -> 36-3039-ND; Supplier2 (none) -> Mouser; Supplier2 link (none) -> http://se.mouser.com/ProductDetail/Keystone-Electronics/303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; Supplier2 part (none) -> 534-3039
- C1: Supplier5 (none) -> RS; Supplier5 link (none) -> http://se.rs-online.com/web/p/tantalum-capacitors/4070047; Supplier5 part (none) -> 407-0047
- C10, C12, C13, C14: Supplier1 Mouser -> AliExpress; Supplier1 link http://se.mouser.com/ProductDetail/AVX/TPSB475K025R0900/?qs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 -> http://www.aliexpress.com/item/Free-shipping-20pcs-B-3528-4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; Supplier1 part 581-TPSB475K025R0900 -> 32456411946; Supplier4 Elfa -> Mouser; Supplier4 link https://www.elfa.se/elfa3~se_sv/elfa/init.do?item=67-700-69 -> http://se.mouser.com/ProductDetail/AVX/TPSB475K025R0900/?qs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; Supplier4 part 67-700-69 -> 581-TPSB475K025R0900; Supplier5 AliExpress -> RS; Supplier5 link http://www.aliexpress.com/item/Free-shipping-20pcs-B-3528-4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 -> http://se.rs-online.com/web/p/tantalum-capacitors/6993349; Supplier5 part 32456411946 -> 699-3349
- C11, C15, C16, C17, C18: Vendor part RR1220P-105-B-T5 -> MCSH31B104K250CT
- C2: Supplier5 Elfa -> RS; Supplier5 link https://www.elfa.se/elfa3~se_sv/elfa/init.do?item=67-700-69 -> http://se.rs-online.com/web/p/tantalum-capacitors/6993349; Supplier5 part 67-700-69 -> 699-3349
- C5, C6: Supplier5 Elfa -> RS; Supplier5 link https://www.elfa.se/elfa3~se_en/elfa/init.do?item=65-721-38 -> http://se.rs-online.com/web/p/ceramic-multilayer-capacitors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; Supplier5 part 65-721-38 -> 723-6616
- C7: Supplier1 link http://se.farnell.com/multicomp/mcsh31b104k250ct/cap-mlcc-x7r-100nf-25v-1206/dp/1856619?ost=1856619 -> http://se.farnell.com/multicomp/mcsh31b104k250ct/cap-mlcc-x7r-100nf-25v-1206/dp/1856619; Vendor part RR1220P-105-B-T5 -> MCSH31B104K250CT
- C8: Supplier1 Mouser -> User specific; Supplier2 Farnell -> (none); Supplier3 Elfa -> (none); Supplier4 Digi-Key -> (none); Supplier5 AliExpress -> (none); Vendor (none) -> User specific
- C9: Supplier1 Mouser -> Farnell; Supplier1 link http://www.mouser.se/ProductDetail/Vishay-Vitramon/VJ1206Y1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 -> http://se.farnell.com/multicomp/mc1206b104k250ct/cap-mlcc-x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; Supplier1 part 77-VJ1206Y104KXXCBC -> 1759312; Supplier2 Farnell -> AliExpress; Supplier2 link http://se.farnell.com/multicomp/mc1206b104k250ct/cap-mlcc-x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 -> http://www.aliexpress.com/item/200pcs-lot-CL31B104KACNNNC-C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; Supplier2 part 1759312 -> 32323646062; Supplier3 Digi-Key -> Mouser; Supplier3 link http://www.digikey.se/short/t4zm2w -> http://www.mouser.se/ProductDetail/Vishay-Vitramon/VJ1206Y1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; Supplier3 part 1276-2742-1-ND -> 77-VJ1206Y104KXXCBC; Supplier4 Elfa -> Digi-Key; Supplier4 link https://www.elfa.se/elfa3~se_en/elfa/init.do?item=65-722-69 -> http://www.digikey.se/short/t4zm2w; Supplier4 part 65-722-69 -> 1276-2742-1-ND; Supplier5 AliExpress -> Elfa; Supplier5 link http://www.aliexpress.com/item/200pcs-lot-CL31B104KACNNNC-C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 -> https://www.elfa.se/elfa3~se_en/elfa/init.do?item=65-755-90; Supplier5 part 32323646062 -> 65-755-90
- JP1, JP3, JP6: Supplier1 link http://se.farnell.com/wurth-elektronik/61300211121/header-2-54mm-pin-tht-vertical/dp/2356153?ost=61300211121 -> http://se.farnell.com/wurth-elektronik/61300211121/header-2-54mm-pin-tht-vertical/dp/2356153; Supplier4 Elfa -> RS; Supplier4 link https://www.elfa.se/elfa3~se_en/elfa/init.do?item=43-004-90 -> http://se.rs-online.com/web/p/pcb-headers/8281581; Supplier4 part 43-004-90 -> 828-1581; Supplier5 (none) -> Elfa; Supplier5 link (none) -> https://www.elfa.se/elfa3~se_en/elfa/init.do?item=43-004-90; Supplier5 part (none) -> 43-004-90; Vendor HARWIN -> Wurth Electronics; Vendor part M20-9993646 -> 61300211121
- JP10, JP4, JP5, JP7: Supplier1 Mouser -> Farnell; Supplier1 link http://www.mouser.com/ProductDetail/Wurth-Electronics/61300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 -> http://se.farnell.com/wurth-elektronik/61300211121/header-2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; Supplier1 part 710-61300211121 -> 2356153; Supplier2 Farnell -> Digi-Key; Supplier2 link http://se.farnell.com/wurth-elektronik/61300211121/header-2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 -> http://www.digikey.se/short/7w149z; Supplier2 part 2356153 -> S1012EC-02-ND; Supplier3 Elfa -> Mouser; Supplier3 link https://www.elfa.se/elfa3~se_en/elfa/init.do?item=43-004-90 -> http://www.mouser.com/ProductDetail/Wurth-Electronics/61300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; Supplier3 part 43-004-90 -> 710-61300211121; Supplier4 Digi-Key -> RS; Supplier4 link http://www.digikey.se/short/7w149z -> http://se.rs-online.com/web/p/pcb-headers/8281581; Supplier4 part S1012EC-02-ND -> 828-1581; Supplier5 (none) -> Elfa; Supplier5 link (none) -> https://www.elfa.se/elfa3~se_en/elfa/init.do?item=43-004-90; Supplier5 part (none) -> 43-004-90; Vendor HARWIN -> Wurth Electronics; Vendor part M20-9993646 -> 61300211121
- JP2, JP8, JP9: Supplier2 Digi-Key -> RS; Supplier2 link http://www.digikey.se/short/7w1485 -> http://se.rs-online.com/web/p/pcb-headers/7457068; Supplier2 part 952-2264-ND -> 745-7068; Supplier3 Mouser -> Digi-Key; Supplier3 link http://www.mouser.com/ProductDetail/3M-Electronic-Solutions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 -> http://www.digikey.se/short/7w1485; Supplier3 part 517-9611036804AR -> 952-2264-ND; Supplier4 Elfa -> Mouser; Supplier4 link https://www.elfa.se/elfa3~se_en/elfa/init.do?item=43-004-91 -> http://www.mouser.com/ProductDetail/3M-Electronic-Solutions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; Supplier4 part 43-004-91 -> 517-9611036804AR; Supplier5 (none) -> Elfa; Supplier5 link (none) -> https://www.elfa.se/elfa3~se_en/elfa/init.do?item=43-004-91; Supplier5 part (none) -> 43-004-91; Vendor part M20-9993646 -> M20-9990346
- L1: Supplier1 link http://se.farnell.com/tdk/mlz2012m4r7wt/inductor-shielded-4-7uh-20/dp/2215656?ost=CBC2012T4R7M&rpsku=CBC2012T4R7M -> http://se.farnell.com/tdk/mlz2012m4r7wt/inductor-shielded-4-7uh-20/dp/2215656
- P1: Supplier2 Mouser -> RS; Supplier2 link http://www.mouser.se/ProductDetail/Harwin/M20-9981045/?qs=%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 -> http://se.rs-online.com/web/p/pcb-headers/6812969; Supplier2 part 855-M20-9981045 -> 681-2969; Supplier3 Digi-Key -> Mouser; Supplier3 link http://www.digikey.se/short/t4z5r3 -> http://www.mouser.se/ProductDetail/Harwin/M20-9981045/?qs=%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; Supplier3 part 952-2129-ND -> 855-M20-9981045; Supplier4 Farnell -> Digi-Key; Supplier4 link http://se.farnell.com/harwin/m20-9981045/board-to-board-con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 -> http://www.digikey.se/short/t4z5r3; Supplier4 part 2127560 -> 952-2129-ND; Supplier5 (none) -> Farnell; Supplier5 link (none) -> http://se.farnell.com/harwin/m20-9981045/board-to-board-con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; Supplier5 part (none) -> 2127560
- P2: Supplier1 Mouser -> RS; Supplier1 link http://www.mouser.se/ProductDetail/Harwin/M20-9981045/?qs=%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 -> http://se.rs-online.com/web/p/pcb-headers/7457046; Supplier1 part 855-M20-9981045 -> 745-7046; Supplier2 Farnell -> Mouser; Supplier2 link http://se.farnell.com/harwin/m20-9981045/board-to-board-con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 -> http://www.mouser.se/ProductDetail/Harwin/M20-9981045/?qs=%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; Supplier2 part 2127560 -> 855-M20-9981045; Supplier3 Elfa -> Digi-Key; Supplier3 link https://www.elfa.se/elfa3~se_en/elfa/init.do?item=43-006-07 -> http://www.digikey.se/short/7w1m89; Supplier3 part 43-006-07 -> 952-2121-ND; Supplier4 Digi-Key -> Farnell; Supplier4 link http://www.digikey.se/short/7w1m89 -> http://se.farnell.com/harwin/m20-9981045/board-to-board-con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; Supplier4 part 952-2121-ND -> 2127560; Supplier5 (none) -> Elfa; Supplier5 link (none) -> https://www.elfa.se/elfa3~se_en/elfa/init.do?item=43-006-07; Supplier5 part (none) -> 43-006-07; Vendor part M20-9981045 -> M20-9980346
- R1: Supplier2 link http://se.farnell.com/welwyn/pcf0805r-150kbt1/resistor-0805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 -> http://se.farnell.com/welwyn/asc0805-150kft5/resistor-anti-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; Supplier2 part 1160270RL -> 2078969; Supplier5 Elfa -> RS; Supplier5 link https://www.elfa.se/elfa3~se_sv/elfa/init.do?item=60-587-70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 -> http://se.rs-online.com/web/p/surface-mount-fixed-resistors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; Supplier5 part 60-587-70 -> 2508365162
- R6, R7, R8, R9: Supplier4 link https://www.elfa.se/elfa3~se_en/elfa/init.do?item=60-255-52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 -> https://www.elfa.se/elfa3~se_en/elfa/init.do?item=60-255-52
- U1: Supplier1 AliExpress -> RS; Supplier1 link http://www.aliexpress.com/item/ICIC-LD1117-LD1117DT33TR-LD1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 -> http://se.rs-online.com/web/p/low-dropout-voltage-regulator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; Supplier1 part 32395965284 -> 686-9252; Supplier3 (none) -> AliExpress; Supplier3 link (none) -> http://www.aliexpress.com/item/ICIC-LD1117-LD1117DT33TR-LD1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; Supplier3 part (none) -> 32395965284
- U2: Supplier1 Mouser -> RS; Supplier1 link http://www.mouser.com/ProductDetail/Texas-Instruments/TPS61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 -> http://se.rs-online.com/web/p/boost-converters/8123619; Supplier1 part 595-TPS61097A-33DBVT -> 812-3619; Supplier2 Farnell -> AliExpress; Supplier2 link http://se.farnell.com/texas-instruments/tps61097-33dbvr/dc-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 -> http://www.aliexpress.com/item/Free-Shipping-5PCS-lot-TPS61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; Supplier2 part 2352441 -> 32369898019; Supplier3 Elfa -> Mouser; Supplier3 link https://www.elfa.se/elfa3~se_en/elfa/init.do?item=73-295-89 -> http://www.mouser.com/ProductDetail/Texas-Instruments/TPS61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; Supplier3 part 73-295-89 -> 595-TPS61097A-33DBVT; Supplier5 (none) -> Farnell; Supplier5 link (none) -> http://se.farnell.com/texas-instruments/tps61097-33dbvr/dc-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; Supplier5 part (none) -> 2352441
- U4: Supplier1 link http://www.ebay.com/itm/171567167962?rmvSB=true -> http://www.ebay.com/itm/171567167962
- U5: Supplier3 Mouser -> RS; Supplier3 link http://www.mouser.com/ProductDetail/3M-Electronic-Solutions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 -> http://se.rs-online.com/web/p/pcb-sockets/4958638; Supplier3 part 517-929975-01-04-RK -> 495-8638; Supplier4 Elfa -> Mouser; Supplier4 link https://www.elfa.se/elfa3~se_en/elfa/init.do?item=43-006-59 -> http://www.mouser.com/ProductDetail/3M-Electronic-Solutions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; Supplier4 part 43-006-59 -> 517-929975-01-04-RK; Supplier5 (none) -> Elfa; Supplier5 link (none) -> https://www.elfa.se/elfa3~se_en/elfa/init.do?item=43-006-59; Supplier5 part (none) -> 43-006-59
- U6: Supplier1 Mouser -> RS; Supplier1 link http://www.mouser.com/Search/ProductDetail.aspx?R=AT25DF512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 -> http://se.rs-online.com/web/p/flash-memory-chips/8228477; Supplier1 part 988-AT25DF512CSSHN-B -> 822-8477; Supplier2 Farnell -> Mouser; Supplier2 link http://se.farnell.com/adesto-technologies/at45db041e-sshn-b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 -> http://www.mouser.com/Search/ProductDetail.aspx?R=AT25DF512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; Supplier2 part 2414322 -> 988-AT25DF512CSSHN-B; Supplier3 Digi-Key -> Farnell; Supplier3 link http://www.digikey.se/short/7wd874 -> http://se.farnell.com/adesto-technologies/at45db041e-sshn-b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; Supplier3 part 1265-1114-1-ND -> 2414322; Supplier4 (none) -> Digi-Key; Supplier4 link (none) -> http://www.digikey.se/short/7wd874; Supplier4 part (none) -> 1265-1114-1-ND
- U7: Supplier1 link http://www.ebay.com/itm/200914924969?rmvSB=true -> http://www.ebay.com/itm/200914924969
- U8: Supplier3 Farnell -> RS; Supplier3 link http://se.farnell.com/silicon-labs/si7021-a20-gm1/temp-fukt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 -> http://se.rs-online.com/web/p/temperature-humidity-sensors/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; Supplier3 part 2473671 -> 865-2328; Supplier4 (none) -> Farnell; Supplier4 link (none) -> http://se.farnell.com/silicon-labs/si7021-a20-gm1/temp-fukt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; Supplier4 part (none) -> 2473671
- U9: Supplier4 Farnell -> RS; Supplier4 link http://se.farnell.com/texas-instruments/tps61221dckt/dc-dc-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 -> http://se.rs-online.com/web/p/boost-converters/8123631; Supplier4 part 2395700 -> 812-3631; Supplier5 (none) -> Farnell; Supplier5 link (none) -> http://se.farnell.com/texas-instruments/tps61221dckt/dc-dc-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; Supplier5 part (none) -> 2395700
